File: 1u_panel-power.kicad_sch (KiCad schematic)
At the start: 39 parts, among them Q1 DMP3050LVT-7, Q2 DMP2240UDM-7, U12 LTC4412, U4 INA226AIDGSR, U5 LTC3525D-3.3

Commit message: Update schematic.
Parts:
- removed C10: GRM155R70J105KA12D, GRM155R70J105KA12D:CAPC1005X55N, symbol GRM155R70J105KA12D:GRM155R70J105KA12D
- removed C15: 22u, 1u_panel:.0805-B-NOSILK, symbol 1u_panel-eagle-import:oresat-rcl_C-EU0805-B-NOSILK
- removed C21: 100n, 1u_panel:.0402-B-NOSILK, symbol 1u_panel-eagle-import:C-EU0402-B-NOSILK
- removed C7: GRM219R60J106KE19D, GRM219R60J106KE19D:CAPC2012X95N, symbol GRM219R60J106KE19D:GRM219R60J106KE19D
- removed CELL2: SPECTROLAB-XTE-SF, 1u_panel:SPECTROLAB-XTE-SF, symbol 1u_panel-eagle-import:SPECTROLAB-XTE-SF
- removed CF1: M55-6021242R, 1u_panel:HARWIN-M55-60X1242R, symbol 1u_panel-eagle-import:SOLAR-BOARD-CONNECTOR
- removed D1, D3: 1N4151WS, 1u_panel:SOD323-R, symbol 1u_panel-eagle-import:DIODE-SOD323-R
- removed D4: GREEN, 1u_panel:LED-0603, symbol 1u_panel-eagle-import:LED-GREEN0603
- removed L1: XFL2010-682MEC, IND_XFL2010_COC, symbol 2025-11-16_06-15-33:XFL2010-682MEC
- removed Q1: DMP3050LVT-7, 1u_panel:SOT23-6, symbol 1u_panel-eagle-import:MOSFET-PCH-SOT23-6
- removed Q2: DMP2240UDM-7, 1u_panel:SOT23-6, symbol 1u_panel-eagle-import:Q-MOSFET-PCH-dual-SOT23-6_MOSFET-PCH-SOT23-6
- removed R14, R20: 0, 1u_panel:.0805-C-NOSILK, symbol 1u_panel-eagle-import:R-US_0805-C-NOSILK
- removed R19, R8: 100k, 1u_panel:.0603-C-NOSILK, symbol 1u_panel-eagle-import:R-US_0603-C-NOSILK
- removed R21: 2.7k, 1u_panel:.0603-C-NOSILK, symbol 1u_panel-eagle-import:R-US_0603-C-NOSILK
- removed R5: 200k, 1u_panel:.0603-C-NOSILK, symbol 1u_panel-eagle-import:R-US_0603-C-NOSILK
- removed TP1, TP11, TP12, TP14, TP16, TP25, TP9: TEST-POINT-LARGE-SQUARE, 1u_panel:1X01, symbol 1u_panel-eagle-import:TEST-POINT-LARGE-SQUARE
- removed U12: LTC4412, 1u_panel:SOT23-6, symbol 1u_panel-eagle-import:LTC4412
- removed U5: LTC3525D-3.3, Package_TO_SOT_SMD:SOT-363_SC-70-6, symbol Regulator_Switching:LTC3525D-3.3
- added J1: PPPC021LFBN-RC, conn-2pin:CONN_PPPC021_SUL, symbol conn-2pin:PPPC021LFBN-RC
- added J2: PPTC051LFBN-RC, CONN5_1LFBN-RC_SUL, symbol conn-5pin:PPTC051LFBN-RC
- added SC1: Solar_Cell, symbol Device:Solar_Cell
Connections:
- net 3.3V: now also J2.1
- net GND: now also J1.2, J2.5, SC1.2 (-)
- net SCL: now also J2.3
- net SDA: now also J2.2
- net VSOLAR: now also R17.1, U4.10 (VIN+), J2.4, SC1.1 (+)
- net at R17.2, U4.8 (VBUS), U4.9 (VIN-): now also J1.1
Other:
- note added: "Output"
- note added: "We will have to make our own footprint depending on the dimensions/pads of our solar cells"
- note removed: "(6.0, 7.2, 8.4) V set by the 2S2P LiPo packs"
- note removed: "0805"
- note removed: "3.3 V SPS"
- note removed: "3.3V power does NOT go through the MPPT"
- note removed: "CTL has internal ground pulldown. ~{SHDN} going low turns on Q1 which pulls CTL high which shuts off the LTC4412 outputs."
- note removed: "DNP FOR FLIGHT"
- note removed: "Ideal diode (w/"off")"
- note removed: "NOTE: SPS is 3.3V output, but power from DEBUG connector is 3.0V (Schottkey drop) directly into 3.3V"
- note removed: "~1.1 V from the cell"
- moved on the sheet: C4, C6, C8, R17, TP24, TP3, U4
