File: 1u_panel.kicad_sch (KiCad schematic)
At the start: 0 parts

Commit message: Update schematic.
Other:
- removed sheet 1u_panel-microcontroller
Changed lines of the file:
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@@
-		)
-	)
-	(sheet
-		(at 25.4 40.64)
-		(size 12.7 3.81)
-		(exclude_from_sim no)
-		(in_bom yes)
-		(on_board yes)
-		(dnp no)
-		(fields_autoplaced yes)
-		(stroke
-			(width 0)
-			(type solid)
-		)
-		(fill
-			(color 0 0 0 0.0000)
-		)
-		(property "Sheetname" "1u_panel-microcontroller"
-			(at 25.4 39.5634 0)
-			(effects
-				(font
-					(size 2 2)
-					(bold yes)
-				)
-				(justify left bottom)
-			)
-		)
-		(property "Sheetfile" "1u_panel-microcontroller.kicad_sch"
-			(at 25.4 45.0346 0)
-			(effects
-				(font
-					(size 1.27 1.27)
-				)
-				(justify left top)
-			)
-		)
-		(instances
-			(project "1u_panel"
-				(path "/115bd2cd-7c08-4b54-867b-a326ee0699c1"
-					(page "2")
-				)
-			)
 		)
 	)
