File: 1u_panel.kicad_pcb (KiCad board)
At the start: 2 copper layers, 83 x 100 mm, 72 parts, among them J2 2-1734592-0, Q1 DMP3050LVT-7, Q2 DMP2240UDM-7, U1 TCAN330GDCNT, U12 LTC4412, U4 INA226AIDGSR, U5 LTC3525D-3.3, U7 STM32F091CCT7, X1 ECS-160-10-36Q-ES-TR

Commit message: Update schematic.
Parts:
- added J1: PPPC021LFBN-RC, conn-2pin:CONN_PPPC021_SUL, F.Cu at (130.6, 75.7)
- added J3: PPTC041LFBN-RC, conn-4pin:CONN_PPTC041LFBN-RC_SUL, F.Cu at (135.8, 70.5)
Connections:
- C4 pad 1: VSOLAR -> V_SOLAR
- C6 pad 1: VSOLAR -> V_SOLAR
- R17 pad 1: Net-(U4-VIN+) -> V_SOLAR
- TP3 pad 1: VSOLAR -> V_SOLAR
- U4 pad 10: Net-(U4-VIN+) -> V_SOLAR

Commit message: MOST RECENT SOLAR LAYOUT
Parts:
- removed C10: GRM155R70J105KA12D, GRM155R70J105KA12D:CAPC1005X55N
- removed C11, C15, C16, C3, C9: 22u, 1u_panel:.0805-B-NOSILK
- removed C21: 100n, 1u_panel:.0402-B-NOSILK
- removed C25, C26, C29, C30, C31: 100n, 1u_panel:.0603-C-NOSILK
- removed C27, C28: 20p, 1u_panel:.0603-C-NOSILK
- removed C7: GRM219R60J106KE19D, GRM219R60J106KE19D:CAPC2012X95N
- removed CELL2: SPECTROLAB-XTE-SF, 1u_panel:SPECTROLAB-XTE-SF
- removed CF1: M55-6021242R, 1u_panel:HARWIN-M55-60X1242R
- removed D1, D3: 1N4151WS, 1u_panel:SOD323-R
- removed D4: GREEN, 1u_panel:LED-0603
- removed D6: AMBER, 1u_panel:LED-0603
- removed J3: PPTC041LFBN-RC, conn-4pin:CONN_PPTC041LFBN-RC_SUL
- removed L1: XFL2010-682MEC, IND_XFL2010_COC:IND_XFL2010_COC
- removed PCB1: ORESAT-SOLAR-BOARD-V4-SPECTROLABS, 1u_panel:ORESAT-SOLAR-BOARD-V4
- removed Q1: DMP3050LVT-7, 1u_panel:SOT23-6
- removed Q2: DMP2240UDM-7, 1u_panel:SOT23-6
- removed R14, R15, R20: 0, 1u_panel:.0805-C-NOSILK
- removed R19, R8: 100k, 1u_panel:.0603-C-NOSILK
- removed R21, R23: 2.7k, 1u_panel:.0603-C-NOSILK
- removed R22: 10k, 1u_panel:.0603-C-NOSILK
- removed R24, R25, R26, R27: 1k/NP, 1u_panel:.0603-C-NOSILK
- removed R5: 200k, 1u_panel:.0603-C-NOSILK
- removed TP1, TP11, TP12, TP13, TP14, TP15, TP16, TP17, TP18, TP19, TP20, TP21, TP22, TP25, TP7, TP8, TP9: TEST-POINT-LARGE-SQUARE, 1u_panel:1X01
- removed U$1: FLIGHMARKERNEW, 1u_panel:FLIGHTMARKER_NEW_BOARDS
- removed U$2, U$3, U$4: FIDUCIAL, 1u_panel:FIDUCIAL_1MM
- removed U1: TCAN330GDCNT, 1u_panel:SOT23-8_TI-DCN
- removed U12: LTC4412, 1u_panel:SOT23-6
- removed U5: LTC3525D-3.3, Package_TO_SOT_SMD:SOT-363_SC-70-6
- removed U7: STM32F091CCT7, 1u_panel:STM32F091C
- removed X1: ECS-160-10-36Q-ES-TR, 1u_panel:CRYSTAL_2.5X2
- J2: value 2-1734592-0 -> PPTC051LFBN-RC; footprint J-TE-2-1734592-0:J-TE-2-1734592-0 -> conn-5pin:CONN5_1LFBN-RC_SUL
- moved R17 124.1 mm to (85.6, 40.4), turned to -90 degrees
- moved TP24 112.2 mm to (105.9, 43.2)
- moved TP3 109.3 mm to (84.8, 48.0)
- moved C8 90.3 mm to (94.4, 39.0), turned to 180 degrees
- moved U4 86.7 mm to (98.0, 43.2), turned to 180 degrees
- moved C6 82.1 mm to (91.7, 45.5), turned to -90 degrees
- moved C4 80.9 mm to (87.4, 45.5), turned to -90 degrees
- moved J1 53.3 mm to (90.0, 41.1), turned to -90 degrees
- moved J2 40.8 mm to (85.7, 30.9)
Connections:
- C4 pad 1: V_SOLAR -> VSOLAR
- C6 pad 1: V_SOLAR -> VSOLAR
- J2 pad 1: Net-(J2-VBUSP-Pad1) -> VSOLAR
- J2 pad 2: Net-(J2-VBUSP-Pad1) -> GND
- J2 pad 3: GND -> 3.3V
- J2 pad 4: unconnected-(J2-DEVICE-D+-Pad4) -> SCL
- J2 pad 5: unconnected-(J2-DEVICE-D--Pad5) -> SDA
- R17 pad 1: V_SOLAR -> VSOLAR
- TP3 pad 1: V_SOLAR -> VSOLAR
- U4 pad 10: V_SOLAR -> VSOLAR
Routing:
- net GND: track 0.00 -> 77.4 mm
- net VSOLAR: track 0.00 -> 31.5 mm
- net SDA: track 0.00 -> 16.3 mm
- net 3.3V: track 0.00 -> 14.6 mm
- net SCL: track 0.00 -> 14.3 mm
- net Net-(U4-VBUS): track 0.00 -> 11.9 mm
- net Net-(U4-ALERT): track 0.00 -> 5.20 mm
Other:
- board outline removed
